File: pcb_formfactor/DifNif.kicad_pcb (KiCad board)
At the start: 2 copper layers, 98.8 x 93 mm, 85 parts, among them J1 DBA-ESDI, J2 PROG, J3 SDCARD_DM3AT-SF-PEJM5, J4 HPLA_PORT, U1 ICE40HX4K-TQ144, U10 74LVC8T245, U11 74LCX07, U12 74VHCT125, U13 Teensy4_1, U14 74LVC8T245, U2 SST26VF080A-104I/SN, U3 APX803S00-29SA-7, U4 AP2114HA-3.3, U5 AP2114HA-1.2, U6 74LVC8T245, U7 74LVC8T245, U8 74LVC8T245, U9 74LVC8T245, X1 ASE-xxxMHz

Commit message: Rev P2: update silkscreen revision
Other:
- board text added: "REV P2 09/26"
- board text removed: "REV P1 11/23"
Changed lines of the file:
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@@
 		)
 	)
-	(gr_text "REV P1\n11/23"
+	(gr_text "REV P2\n09/26"
 		(at 112.3 42 0)
 		(layer "F.SilkS")

Commit message: Rev P2: credit line, refilled pours, fab files
Other:
- board text added: "Tube Time: Design, PCB, Verilog Bitsavers: Documentation, Testing Ardent Tool of Capitalism: More documentation thenetworkinglab: Rev P2 changes SHOUTS TO The Twitch Stream Folks The Retro Tech Crew IBMMuseum Tomáš"
- board text removed: "Tube Time: Design, PCB, Verilog Bitsavers: Documentation, Testing Ardent Tool of Capitalism: More documentation SHOUTS TO The Twitch Stream Folks The Retro Tech Crew IBMMuseum Tomáš"
Changed lines of the file:
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@@
 		(layer "Dwgs.User")
+	)
+	(gr_line
+		(start 91.2 44.36)
+		(end 99.4 44.36)
+		(stroke
+			(width 0.1)
+			(type solid)
+		)
+		(layer "Edge.Cuts")
 	)
 	(gr_arc
@@
 	)
 	(gr_line
+		(start 91.2 129.8)
+		(end 91.2 44.36)
+		(stroke
+			(width 0.1)
+			(type solid)
+		)
+		(layer "Edge.Cuts")
+	)
+	(gr_line
 		(start 92.4 131)
 		(end 190 131)
@@
 	)
 	(gr_line
-		(start 91.2 129.8)
-		(end 91.2 44.36)
-		(stroke
-			(width 0.1)
-			(type solid)
-		)
-		(layer "Edge.Cuts")
-	)
-	(gr_line
-		(start 91.2 44.36)
-		(end 99.4 44.36)
-		(stroke
-			(width 0.1)
-			(type solid)
-		)
-		(layer "Edge.Cuts")
-	)
-	(gr_arc
-		(start 99.4 44.36)
-		(mid 99.9 43.86)
-		(end 99.4 43.36)
-		(stroke
-			(width 0.1)
-			(type solid)
-		)
-		(layer "Edge.Cuts")
-	)
-	(gr_line
 		(start 99.4 43.36)
 		(end 91.2 43.36)
+		(stroke
+			(width 0.1)
+			(type solid)
+		)
+		(layer "Edge.Cuts")
+	)
+	(gr_arc
+		(start 99.4 43.36)
+		(mid 99.9 43.86)
+		(end 99.4 44.36)
 		(stroke
 			(width 0.1)
@@
 		)
 	)
-	(gr_text "Tube Time: Design, PCB, Verilog\nBitsavers: Documentation, Testing\nArdent Tool of Capitalism: More documentation\nSHOUTS TO\nThe Twitch Stream Folks\nThe Retro Tech Crew\nIBMMuseum\nTomáš\n"
-		(at 157.1 69.4 0)
+	(gr_text "Tube Time: Design, PCB, Verilog\nBitsavers: Documentation, Testing\nArdent Tool of Capitalism: More documentation\nthenetworkinglab: Rev P2 changes\nSHOUTS TO\nThe Twitch Stream Folks\nThe Retro Tech Crew\nIBMMuseum\nTomáš\n"
+		(at 157.1 70.4 0)
 		(layer "B.SilkS")
 		(effects
