File: pcb_formfactor/DifNifBus.kicad_sch (KiCad schematic)
At the start: 24 parts, among them J1 DBA-ESDI, U10 74LVC4245, U11 74LCX07, U12 74VHCT125, U14 74LVC4245, U6 74LVC4245, U7 74LVC4245, U8 74LVC4245, U9 74LVC4245

Commit message: Rev P2 schematic: CHRESET fix, 74LVC8T245, -CD SFDBK, debug header
Parts:
- U10, U14, U6, U7, U8, U9: value 74LVC4245 -> 74LVC8T245; Mouser 771-74LVC4245APW-T -> 595-SN74LVC8T245PWR
Connections:
- net ~{CHRESET}_5V is gone; now on net CHRESET_5V: J1.b14 (Pin_b14), U8.14 (B7)
- net GND: no longer U12.13
- net ~{CD_SFDBK}_5V: now reaches U12.11
- net ~{CD_SFDBK}_5V: now also J1.b8 (Pin_b8)
- new net ~{CD_SFDBK}: U12.13
- no-connect marks 6 -> 4
Changed lines of the file:
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@@
   )
   (no_connect (at 48.26 78.74))
-  (no_connect (at 60.96 48.26))
   (no_connect (at 60.96 38.1))
   (no_connect (at 48.26 96.52))
   (no_connect (at 48.26 76.2))
-  (no_connect (at 252.73 140.97))
   (bus_entry (at 185.42 124.46) (size -2.54 -2.54)
     (stroke (width 0) (type default) (color 0 0 0 0))
@@
     (stroke (width 0) (type default) (color 0 0 0 0))
   )
+  (wire (pts (xy 260.35 147.32) (xy 260.35 151.13))
+    (stroke (width 0) (type default) (color 0 0 0 0))
+  )
+  (wire (pts (xy 260.35 151.13) (xy 264.16 151.13))
+    (stroke (width 0) (type default) (color 0 0 0 0))
+  )
+  (hierarchical_label "~{CD_SFDBK}" (shape input) (at 264.16 151.13 0)
+    (effects (font (size 1.27 1.27)) (justify left))
+  )
+  (wire (pts (xy 252.73 140.97) (xy 245.11 140.97))
+    (stroke (width 0) (type default) (color 0 0 0 0))
+  )
+  (label "~{CD_SFDBK}_5V" (at 245.11 140.97 180)
+    (effects (font (size 1.27 1.27)) (justify right bottom))
+  )
+  (wire (pts (xy 60.96 48.26) (xy 74.93 48.26))
+    (stroke (width 0) (type default) (color 0 0 0 0))
+  )
+  (label "~{CD_SFDBK}_5V" (at 74.93 48.26 180)
+    (effects (font (size 1.27 1.27)) (justify right bottom))
+  )
   (wire (pts (xy 31.75 111.76) (xy 48.26 111.76))
     (stroke (width 0) (type default) (color 0 0 0 0))
@@
     (effects (font (size 1.27 1.27)) (justify left bottom))
   )
-  (label "~{CHRESET}_5V" (at 92.71 137.16 0)
+  (label "CHRESET_5V" (at 92.71 137.16 0)
     (effects (font (size 1.27 1.27)) (justify left bottom))
   )
@@
     (effects (font (size 1.27 1.27)) (justify right bottom))
   )
-  (label "~{CHRESET}_5V" (at 74.93 63.5 180)
+  (label "CHRESET_5V" (at 74.93 63.5 180)
     (effects (font (size 1.27 1.27)) (justify right bottom))
   )
@@
       (effects (font (size 1.27 1.27)) (justify left))
     )
-    (property "Value" "74LVC4245" (id 1) (at 129.0194 161.29 0)
+    (property "Value" "74LVC8T245" (id 1) (at 129.0194 161.29 0)
       (effects (font (size 1.27 1.27)) (justify left))
     )
@@
       (effects (font (size 1.27 1.27)) hide)
     )
-    (property "Mouser" "771-74LVC4245APW-T" (id 4) (at 109.22 163.83 0)
+    (property "Mouser" "595-SN74LVC8T245PWR" (id 4) (at 109.22 163.83 0)
       (effects (font (size 1.27 1.27)) hide)
     )
@@
       (effects (font (size 1.27 1.27)) (justify left))
     )
-    (property "Value" "74LVC4245" (id 1) (at 202.6794 72.39 0)
+    (property "Value" "74LVC8T245" (id 1) (at 202.6794 72.39 0)
       (effects (font (size 1.27 1.27)) (justify left))
     )
@@
       (effects (font (size 1.27 1.27)) hide)
     )
-    (property "Mouser" "771-74LVC4245APW-T" (id 4) (at 182.88 74.93 0)
+    (property "Mouser" "595-SN74LVC8T245PWR" (id 4) (at 182.88 74.93 0)
       (effects (font (size 1.27 1.27)) hide)
     )
@@
       (effects (font (size 1.27 1.27)) (justify left))
     )
-    (property "Value" "74LVC4245" (id 1) (at 127.7494 66.04 0)
+    (property "Value" "74LVC8T245" (id 1) (at 127.7494 66.04 0)
       (effects (font (size 1.27 1.27)) (justify left))
     )
@@
       (effects (font (size 1.27 1.27)) hide)
     )
-    (property "Mouser" "771-74LVC4245APW-T" (id 4) (at 107.95 68.58 0)
+    (property "Mouser" "595-SN74LVC8T245PWR" (id 4) (at 107.95 68.58 0)
       (effects (font (size 1.27 1.27)) hide)
     )
@@
       (effects (font (size 1.27 1.27)) (justify left))
     )
-    (property "Value" "74LVC4245" (id 1) (at 127.7494 21.59 0)
+    (property "Value" "74LVC8T245" (id 1) (at 127.7494 21.59 0)
       (effects (font (size 1.27 1.27)) (justify left))
     )
@@
       (effects (font (size 1.27 1.27)) hide)
     )
-    (property "Mouser" "771-74LVC4245APW-T" (id 4) (at 107.95 24.13 0)
+    (property "Mouser" "595-SN74LVC8T245PWR" (id 4) (at 107.95 24.13 0)
       (effects (font (size 1.27 1.27)) hide)
     )
@@
     (pin "9")
   )
-  (symbol (lib_id "power:GND") (at 260.35 147.32 0) (unit 1)
-    (in_bom yes) (on_board yes)
-    (property "Reference" "#PWR05" (id 0) (at 260.35 153.67 0)
-      (effects (font (size 1.27 1.27)) hide)
-    )
-    (property "Value" "GND" (id 1) (at 260.477 151.7142 0)
-      (effects (font (size 1.27 1.27)) hide)
-    )
-    (property "Footprint" "" (id 2) (at 260.35 147.32 0)
-      (effects (font (size 1.27 1.27)) hide)
-    )
-    (property "Datasheet" "" (id 3) (at 260.35 147.32 0)
-      (effects (font (size 1.27 1.27)) hide)
-    )
-    (pin "1")
-  )
   (symbol (lib_id "74xx:74LCX07") (at 260.35 102.87 180) (unit 4)
     (in_bom yes) (on_board yes)
@@
       (effects (font (size 1.27 1.27)) (justify left))
     )
-    (property "Value" "74LVC4245" (id 1) (at 127.7494 114.3 0)
+    (property "Value" "74LVC8T245" (id 1) (at 127.7494 114.3 0)
       (effects (font (size 1.27 1.27)) (justify left))
     )
@@
       (effects (font (size 1.27 1.27)) hide)
     )
-    (property "Mouser" "771-74LVC4245APW-T" (id 4) (at 107.95 116.84 0)
+    (property "Mouser" "595-SN74LVC8T245PWR" (id 4) (at 107.95 116.84 0)
       (effects (font (size 1.27 1.27)) hide)
     )
@@
       (effects (font (size 1.27 1.27)) (justify left))
     )
-    (property "Value" "74LVC4245" (id 1) (at 202.6794 25.4 0)
+    (property "Value" "74LVC8T245" (id 1) (at 202.6794 25.4 0)
       (effects (font (size 1.27 1.27)) (justify left))
     )
@@
       (effects (font (size 1.27 1.27)) hide)
     )
-    (property "Mouser" "771-74LVC4245APW-T" (id 4) (at 182.88 27.94 0)
+    (property "Mouser" "595-SN74LVC8T245PWR" (id 4) (at 182.88 27.94 0)
       (effects (font (size 1.27 1.27)) hide)
     )

Commit message: Drive -CD SFDBK push-pull from U12 pin 12; ignore KiCad working files
Connections:
- net GND: now also U12.13; no longer U12.12
- net ~{CD_SFDBK}: now also U12.12; no longer U12.13
Changed lines of the file:
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@@
     (stroke (width 0) (type default) (color 0 0 0 0))
   )
-  (wire (pts (xy 260.35 147.32) (xy 260.35 151.13))
-    (stroke (width 0) (type default) (color 0 0 0 0))
-  )
-  (wire (pts (xy 260.35 151.13) (xy 264.16 151.13))
-    (stroke (width 0) (type default) (color 0 0 0 0))
-  )
-  (hierarchical_label "~{CD_SFDBK}" (shape input) (at 264.16 151.13 0)
+  (hierarchical_label "~{CD_SFDBK}" (shape input) (at 271.78 148.59 0)
     (effects (font (size 1.27 1.27)) (justify left))
   )
@@
     (effects (font (size 1.27 1.27)) (justify right bottom))
   )
+  (wire (pts (xy 269.24 146.05) (xy 269.24 148.59))
+    (stroke (width 0) (type default) (color 0 0 0 0))
+  )
+  (wire (pts (xy 269.24 148.59) (xy 271.78 148.59))
+    (stroke (width 0) (type default) (color 0 0 0 0))
+  )
   (wire (pts (xy 31.75 111.76) (xy 48.26 111.76))
     (stroke (width 0) (type default) (color 0 0 0 0))
@@
     (pin "1")
   )
-  (symbol (lib_id "power:GND") (at 269.24 146.05 0) (unit 1)
+  (symbol (lib_id "power:GND") (at 260.35 147.32 0) (unit 1)
     (in_bom yes) (on_board yes)
-    (property "Reference" "#PWR06" (id 0) (at 269.24 152.4 0)
+    (property "Reference" "#PWR06" (id 0) (at 260.35 153.67 0)
       (effects (font (size 1.27 1.27)) hide)
     )
-    (property "Value" "GND" (id 1) (at 269.367 150.4442 0)
+    (property "Value" "GND" (id 1) (at 260.477 151.7142 0)
       (effects (font (size 1.27 1.27)) hide)
     )
-    (property "Footprint" "" (id 2) (at 269.24 146.05 0)
+    (property "Footprint" "" (id 2) (at 260.35 147.32 0)
       (effects (font (size 1.27 1.27)) hide)
     )
-    (property "Datasheet" "" (id 3) (at 269.24 146.05 0)
+    (property "Datasheet" "" (id 3) (at 260.35 147.32 0)
       (effects (font (size 1.27 1.27)) hide)
     )

Commit message: Relabel level-shifter symbol as 74LVC8T245; note Model 70 socket is unkeyed
Parts:
- U10, U14, U6, U7, U8, U9: symbol logic:74LVC4245 -> logic:74LVC8T245
Changed lines of the file:
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@@
     (pin "2")
   )
-  (symbol (lib_id "logic:74LVC4245") (at 109.22 163.83 0) (unit 1)
+  (symbol (lib_id "logic:74LVC8T245") (at 109.22 163.83 0) (unit 1)
     (in_bom yes) (on_board yes) (fields_autoplaced)
     (property "Reference" "U9" (id 0) (at 129.0194 158.75 0)
@@
     (pin "9")
   )
-  (symbol (lib_id "logic:74LVC4245") (at 182.88 74.93 0) (unit 1)
+  (symbol (lib_id "logic:74LVC8T245") (at 182.88 74.93 0) (unit 1)
     (in_bom yes) (on_board yes) (fields_autoplaced)
     (property "Reference" "U14" (id 0) (at 202.6794 69.85 0)
@@
     (pin "1")
   )
-  (symbol (lib_id "logic:74LVC4245") (at 107.95 68.58 0) (unit 1)
+  (symbol (lib_id "logic:74LVC8T245") (at 107.95 68.58 0) (unit 1)
     (in_bom yes) (on_board yes) (fields_autoplaced)
     (property "Reference" "U7" (id 0) (at 127.7494 63.5 0)
@@
     (pin "2")
   )
-  (symbol (lib_id "logic:74LVC4245") (at 107.95 24.13 0) (unit 1)
+  (symbol (lib_id "logic:74LVC8T245") (at 107.95 24.13 0) (unit 1)
     (in_bom yes) (on_board yes) (fields_autoplaced)
     (property "Reference" "U6" (id 0) (at 127.7494 19.05 0)
@@
     (pin "1")
   )
-  (symbol (lib_id "logic:74LVC4245") (at 107.95 116.84 0) (unit 1)
+  (symbol (lib_id "logic:74LVC8T245") (at 107.95 116.84 0) (unit 1)
     (in_bom yes) (on_board yes) (fields_autoplaced)
     (property "Reference" "U8" (id 0) (at 127.7494 111.76 0)
@@
     (pin "9")
   )
-  (symbol (lib_id "logic:74LVC4245") (at 182.88 27.94 0) (unit 1)
+  (symbol (lib_id "logic:74LVC8T245") (at 182.88 27.94 0) (unit 1)
     (in_bom yes) (on_board yes) (fields_autoplaced)
     (property "Reference" "U10" (id 0) (at 202.6794 22.86 0)
